Commit message: Fixed compilation issues. Ready for hardware testing

File: install/swarm_bot/share/swarm_bot/description/inertial_macros.xacro (robot description, xacro)
@@ -1,33 +1 @@
-<?xml version="1.0"?>
-<robot xmlns:xacro="http://www.ros.org/wiki/xacro" >
-    <!-- Specify some standard inertial calculations https://en.wikipedia.org/wiki/List_of_moments_of_inertia -->
-    <!-- From https://github.com/joshnewans/articubot_one/blob/d5aa5e9bc9039073c0d8fd7fe426e170be79c087/description/inertial_macros.xacro -->
-    <!-- These make use of xacro's mathematical functionality -->
-    <xacro:macro name="inertial_sphere" params="mass radius *origin">
-        <inertial>
-            <xacro:insert_block name="origin"/>
-            <mass value="${mass}" />
-            <inertia ixx="${(2/5) * mass * (radius*radius)}" ixy="0.0" ixz="0.0"
-                    iyy="${(2/5) * mass * (radius*radius)}" iyz="0.0"
-                    izz="${(2/5) * mass * (radius*radius)}" />
-        </inertial>
-    </xacro:macro>
-    <xacro:macro name="inertial_box" params="mass x y z *origin">
-        <inertial>
-            <xacro:insert_block name="origin"/>
-            <mass value="${mass}" />
-            <inertia ixx="${(1/12) * mass * (y*y+z*z)}" ixy="0.0" ixz="0.0"
-                    iyy="${(1/12) * mass * (x*x+z*z)}" iyz="0.0"
-                    izz="${(1/12) * mass * (x*x+y*y)}" />
-        </inertial>
-    </xacro:macro>
-    <xacro:macro name="inertial_cylinder" params="mass length radius *origin">
-        <inertial>
-            <xacro:insert_block name="origin"/>
-            <mass value="${mass}" />
-            <inertia ixx="${(1/12) * mass * (3*radius*radius + length*length)}" ixy="0.0" ixz="0.0"
-                    iyy="${(1/12) * mass * (3*radius*radius + length*length)}" iyz="0.0"
-                    izz="${(1/2) * mass * (radius*radius)}" />
-        </inertial>
-    </xacro:macro>
-</robot>
+/home/ubuntu/Documents/swarm/ros/src/swarm_bot/description/inertial_macros.xacro

File: install/swarm_bot/share/swarm_bot/description/robot.urdf.xacro (robot description, xacro)
@@ -1,13 +1 @@
-<?xml version="1.0"?>
-<robot xmlns:xacro="http://www.ros.org/wiki/xacro"  name="robot">
-<!-- ROS2 control is definitely better for the real robot but can be a little funkier in Gazebo -->
-  <xacro:arg name="use_ros2_control" default="true" />
-  <xacro:include filename="robot_core.xacro" />
-  <xacro:if value="$(arg use_ros2_control)">
-    <xacro:include filename="ros2_control.xacro" />
-  </xacro:if>
-  <xacro:unless value="$(arg use_ros2_control)">
-    <xacro:include filename="gazebo_control.xacro" />
-  </xacro:unless>
-  <xacro:include filename="camera.xacro" />
-</robot>
+/home/ubuntu/Documents/swarm/ros/src/swarm_bot/description/robot.urdf.xacro

File: install/swarm_bot/share/swarm_bot/description/robot_core.xacro (robot description, xacro)
@@ -1,141 +1 @@
-<?xml version="1.0"?>
-<robot xmlns:xacro="http://www.ros.org/wiki/xacro"  name="robot">
-  <xacro:include filename="inertial_macros.xacro" />
-  <material name="black">
-    <color rgba="0 0 0 1"/>
-  </material>
-  <material name="white">
-    <color rgba="1 1 1 1"/>
-  </material>
-  <material name="orange">
-    <color rgba="1 0.5 0 1"/>
-  </material>
-  <material name="blue">
-    <color rgba="0 0 1 1"/>
-  </material>
-  <material name="red">
-    <color rgba="1 0 0 1"/>
-  </material>
-  <material name="green">
-    <color rgba="0 1 0 1"/>
-  </material>
-  <!-- BASE LINK -->
-  <!-- Set to be the center of the two drive wheels -->
-  <link name="base_link">
-  </link>
-  <!-- CHASSIS LINK -->
-  <joint name="chassis_joint" type="fixed">
-    <parent link="base_link"/>
-    <child link="chassis"/>
-    <origin xyz="0 0 0.025" />
-  </joint>
-  <link name="chassis">
-    <!-- Cylinder with r=120mm, h=50mm (ASSUMPTION) -->
-    <visual>
-      <geometry>
-        <cylinder length="0.05" radius="0.12"/>
-      </geometry>
-      <material name="white"/>
-    </visual>
-    <collision>
-      <geometry>
-        <cylinder length="0.05" radius="0.12"/>
-      </geometry>
-    </collision>
-    <!-- Mass=0.5kg (ASSUMPTION) -->
-    <xacro:inertial_cylinder mass="0.5" length="0.05" radius="0.12">
-      <!-- Not sure if this is correct -->
-      <origin xyz="0 0 0.025" rpy="0 0 0"/>
-    </xacro:inertial_cylinder>
-  </link>
-  <gazebo reference="chassis">
-    <material>Gazebo/White</material>
-  </gazebo>
-  <!-- LEFT WHEEL LINK -->
-  <joint name="left_wheel_joint" type="continuous">
-    <parent link="base_link"/>
-    <child link="left_wheel"/>
-    <origin xyz="0 0.122 0" rpy="-${pi/2} 0 0"/>
-    <axis xyz="0 0 1"/>
-  </joint>
-  <link name="left_wheel">
-    <!-- Cylinder with r=30mm, h=8mm (FROM WEBSITE) -->
-    <visual>
-      <geometry>
-        <cylinder length="0.008" radius="0.03"/>
-      </geometry>
-      <material name="blue"/>
-    </visual>
-    <collision>
-      <geometry>
-        <cylinder length="0.008" radius="0.03"/>
-      </geometry>
-    </collision>
-    <!-- Mass=0.1kg (ASSUMPTION) -->
-    <xacro:inertial_cylinder mass="0.1" length="0.008" radius="0.03">
-      <origin xyz="0 0 0" rpy="0 0 0"/>
-    </xacro:inertial_cylinder>
-  </link>
-  <gazebo reference="left_wheel">
-    <material>Gazebo/Blue</material>
-  </gazebo>
-  <!-- RIGHT WHEEL LINK -->
-  <joint name="right_wheel_joint" type="continuous">
-    <parent link="base_link"/>
-    <child link="right_wheel"/>
-    <origin xyz="0 -0.122 0" rpy="${pi/2} 0 0"/>
-    <axis xyz="0 0 -1"/>
-  </joint>
-  <link name="right_wheel">
-    <!-- Cylinder with r=30mm, h=8mm (FROM WEBSITE) -->
-    <visual>
-      <geometry>
-        <cylinder length="0.008" radius="0.03"/>
-      </geometry>
-      <material name="blue"/>
-    </visual>
-    <collision>
-      <geometry>
-        <cylinder length="0.008" radius="0.03"/>
-      </geometry>
-    </collision>
-    <!-- Mass=0.1kg (ASSUMPTION) -->
-    <xacro:inertial_cylinder mass="0.1" length="0.008" radius="0.03">
-      <origin xyz="0 0 0" rpy="0 0 0"/>
-    </xacro:inertial_cylinder>
-  </link>
-  <gazebo reference="right_wheel">
-    <material>Gazebo/Blue</material>
-  </gazebo>
-  <!-- CASTER WHEEL LINK -->
-  <!-- Frictionless ball that does not rotate -->
-  <joint name="caster_wheel_joint" type="fixed">
-    <parent link="chassis"/>
-    <child link="caster_wheel"/>
-    <origin xyz="-0.0875 0 -0.03"/>
-  </joint>
-  <link name="caster_wheel">
-    <!-- Sphere with r=25mm (ASSUMPTION) -->
-    <visual>
-      <geometry>
-        <sphere radius="0.025"/>
-      </geometry>
-      <material name="red"/>
-    </visual>
-    <collision>
-      <geometry>
-        <sphere radius="0.025"/>
-      </geometry>
-    </collision>
-    <!-- Mass=0.1kg (ASSUMPTION) -->
-    <xacro:inertial_sphere mass="0.1" radius="0.025">
-      <origin xyz="0 0 0" rpy="0 0 0"/>
-    </xacro:inertial_sphere>
-  </link>
-  <!-- No friction -->
-  <gazebo reference="caster_wheel">
-    <material>Gazebo/Red</material>
-    <mu1>0.001</mu1>
-    <mu2>0.001</mu2>
-  </gazebo>
-</robot>
+/home/ubuntu/Documents/swarm/ros/src/swarm_bot/description/robot_core.xacro

File: install/swarm_bot/share/swarm_bot/description/ros2_control.xacro (robot description, xacro)
@@ -1,29 +1 @@
-<?xml version="1.0"?>
-<robot xmlns:xacro="http://www.ros.org/wiki/xacro">
-  <ros2_control name="GazeboSystem" type="system">
-    <hardware>
-      <plugin>gazebo_ros2_control/GazeboSystem</plugin>
-    </hardware>
-    <joint name="left_wheel_joint">
-      <command_interface name="velocity">
-        <param name="min">-10</param>
-        <param name="max">10</param>
-      </command_interface>
-      <state_interface name="velocity" />
-      <state_interface name="position" />
-    </joint>
-    <joint name="right_wheel_joint">
-      <command_interface name="velocity">
-        <param name="min">-10</param>
-        <param name="max">10</param>
-      </command_interface>
-      <state_interface name="velocity" />
-      <state_interface name="position" />
-    </joint>
-  </ros2_control>
-  <gazebo>
-    <plugin name="gazebo_ros2_control" filename="libgazebo_ros2_control.so">
-      <parameters>$(find swarm_bot)/config/robot_controllers.yaml</parameters>
-    </plugin>
-  </gazebo>
-</robot>
+/home/ubuntu/Documents/swarm/ros/src/swarm_bot/description/ros2_control.xacro
