Commit message: Added simple Gazebo simulation and environment

File: ros/src/swarm_bot/description/robot.urdf.xacro (robot description, xacro)
@@ -2,3 +2,4 @@
 <robot xmlns:xacro="http://www.ros.org/wiki/xacro"  name="robot">
   <xacro:include filename="robot_core.xacro" />
+  <xacro:include filename="gazebo_control.xacro" />
 </robot>

File: ros/src/swarm_bot/description/robot_core.xacro (robot description, xacro)
@@ -46,4 +46,7 @@
     </xacro:inertial_cylinder>
   </link>
+  <gazebo reference="chassis">
+    <material>Gazebo/White</material>
+  </gazebo>
   <!-- LEFT WHEEL LINK -->
   <joint name="left_wheel_joint" type="continuous">
@@ -71,4 +74,7 @@
     </xacro:inertial_cylinder>
   </link>
+  <gazebo reference="left_wheel">
+    <material>Gazebo/Blue</material>
+  </gazebo>
   <!-- RIGHT WHEEL LINK -->
   <joint name="right_wheel_joint" type="continuous">
@@ -96,4 +102,7 @@
     </xacro:inertial_cylinder>
   </link>
+  <gazebo reference="right_wheel">
+    <material>Gazebo/Blue</material>
+  </gazebo>
   <!-- CASTER WHEEL LINK -->
   <!-- Frictionless ball that does not rotate -->
@@ -121,3 +130,8 @@
     </xacro:inertial_sphere>
   </link>
+  <gazebo reference="caster_wheel">
+    <material>Gazebo/Red</material>
+    <mu1>0.001</mu1>
+    <mu2>0.001</mu2>
+  </gazebo>
 </robot>

Commit message: Switched control to ros2_control and set up joystick

File: ros/src/swarm_bot/description/robot.urdf.xacro (robot description, xacro)
@@ -1,6 +1,13 @@
 <?xml version="1.0"?>
 <robot xmlns:xacro="http://www.ros.org/wiki/xacro"  name="robot">
+<!-- ROS2 control is definitely better for the real robot but can be a little funkier in Gazebo -->
+  <xacro:arg name="use_ros2_control" default="true" />
   <xacro:include filename="robot_core.xacro" />
-  <xacro:include filename="gazebo_control.xacro" />
+  <xacro:if value="$(arg use_ros2_control)">
+    <xacro:include filename="ros2_control.xacro" />
+  </xacro:if>
+  <xacro:unless value="$(arg use_ros2_control)">
+    <xacro:include filename="gazebo_control.xacro" />
+  </xacro:unless>
   <xacro:include filename="camera.xacro" />
 </robot>

File: ros/src/swarm_bot/description/robot_core.xacro (robot description, xacro)
@@ -16,4 +16,7 @@
   <material name="red">
     <color rgba="1 0 0 1"/>
+  </material>
+  <material name="green">
+    <color rgba="0 1 0 1"/>
   </material>
   <!-- BASE LINK -->

Commit message: MAP MADE WITH LIDAR WORKS

File: ros/src/swarm_bot/description/robot.urdf.xacro (robot description, xacro)
@@ -11,3 +11,4 @@
   </xacro:unless>
   <xacro:include filename="camera.xacro" />
+  <xacro:include filename="lidar.xacro" />
 </robot>

File: ros/src/swarm_bot/description/robot_core.xacro (robot description, xacro)
@@ -23,4 +23,12 @@
   <!-- Set to be the center of the two drive wheels -->
   <link name="base_link">
+  </link>
+  <!-- BASE FOOTPRINT LINK -->
+  <joint name="base_footprint_joint" type="fixed">
+  	<parent link="base_link"/>
+  	<child link="base_footprint"/>
+  	<origin xyz="0 0 0" rpy="0 0 0"/>
+  </joint>
+  <link name="base_footprint">
   </link>
   <!-- CHASSIS LINK -->
