Commit message: Fixed wheel orientation of robot
Some changes to theoretically support ball tracking

File: ros/src/swarm_bot/description/camera.xacro (robot description, xacro)
@@ -4,5 +4,5 @@
     <parent link="chassis"/>
     <child link="camera_link"/>
-    <origin xyz="0.08 0 0.025" />
+    <origin xyz="0.08 0 0.025" rpy="0 0.005 0" />
   </joint>
   <link name="camera_link">

File: ros/src/swarm_bot/description/robot_core.xacro (robot description, xacro)
@@ -85,5 +85,5 @@
     <child link="right_wheel"/>
     <origin xyz="0 -0.122 0" rpy="${pi/2} 0 0"/>
-    <axis xyz="0 0 1"/>
+    <axis xyz="0 0 -1"/>
   </joint>
   <link name="right_wheel">

Commit message: Added simulated IMU into Gazebo

File: ros/src/swarm_bot/description/camera.xacro (robot description, xacro)
@@ -1,4 +1,4 @@
 <?xml version="1.0"?>
-<robot xmlns:xacro="http://www.ros.org/wiki/xacro"  name="robot">
+<robot xmlns:xacro="http://www.ros.org/wiki/xacro" name="robot">
   <joint name="camera_joint" type="fixed">
     <parent link="chassis"/>
@@ -7,10 +7,10 @@
   </joint>
   <link name="camera_link">
-    <!-- Cylinder with r=20mm, h=5mm (ASSUMPTION) -->
+    <!-- Box with dimensions 50mm x 30mm x 30mm -->
     <visual>
       <geometry>
         <box size="0.05 0.03 0.03" />
       </geometry>
-      <material name="green"/>
+      <material name="blue"/>
     </visual>
   </link>

File: ros/src/swarm_bot/description/robot.urdf.xacro (robot description, xacro)
@@ -11,3 +11,4 @@
   </xacro:unless>
   <xacro:include filename="camera.xacro" />
+  <xacro:include filename="imu.xacro" />
 </robot>

Commit message: Added stereo camera

File: ros/src/swarm_bot/description/camera.xacro (robot description, xacro)
@@ -1,10 +1,11 @@
 <?xml version="1.0"?>
 <robot xmlns:xacro="http://www.ros.org/wiki/xacro" name="robot">
-  <joint name="camera_joint" type="fixed">
+  <!-- Left Camera -->
+  <joint name="left_camera_joint" type="fixed">
     <parent link="chassis"/>
-    <child link="camera_link"/>
-    <origin xyz="0.08 0 0.025" rpy="0 0.005 0" />
+    <child link="left_camera_link"/>
+    <origin xyz="0.08 -0.05 0.025" rpy="0 0.005 0" />
   </joint>
-  <link name="camera_link">
+  <link name="left_camera_link">
     <!-- Box with dimensions 50mm x 30mm x 30mm -->
     <visual>
@@ -15,13 +16,13 @@
     </visual>
   </link>
-  <joint name="camera_optical_joint" type="fixed">
-    <parent link="camera_link"/>
-    <child link="camera_link_optical"/>
-    <origin xyz="0.08 0 0.025" rpy="${-pi/2} 0 ${-pi/2}" />
+  <joint name="left_camera_optical_joint" type="fixed">
+    <parent link="left_camera_link"/>
+    <child link="left_camera_link_optical"/>
+    <origin xyz="0 0 0" rpy="${-pi/2} 0 ${-pi/2}" />
   </joint>
-  <link name="camera_link_optical"></link>
-  <gazebo reference="camera_link">
+  <link name="left_camera_link_optical"></link>
+  <gazebo reference="left_camera_link">
     <material>Gazebo/Green</material>
-    <sensor name="camera" type="camera">
+    <sensor name="left_camera" type="camera">
       <pose>0 0 0 0 0 0</pose>
       <visualize>true</visualize>
@@ -39,7 +40,52 @@
         </clip>
       </camera>
-      <plugin name="camera_controller" filename="libgazebo_ros_camera.so">
-        <!-- Note that this is associated with the optical link, not the simulated link -->
-        <frame_name>camera_link_optical</frame_name>
+      <plugin name="left_camera_controller" filename="libgazebo_ros_camera.so">
+        <image_topic_name>left_camera/image_raw</image_topic_name>
+        <frame_name>left_camera_link_optical</frame_name>
+      </plugin>
+    </sensor>
+  </gazebo>
+  <!-- Right Camera -->
+  <joint name="right_camera_joint" type="fixed">
+    <parent link="chassis"/>
+    <child link="right_camera_link"/>
+    <origin xyz="0.08 0.05 0.025" rpy="0 0.005 0" />
+  </joint>
+  <link name="right_camera_link">
+    <!-- Box with dimensions 50mm x 30mm x 30mm -->
+    <visual>
+      <geometry>
+        <box size="0.05 0.03 0.03" />
+      </geometry>
+      <material name="blue"/>
+    </visual>
+  </link>
+  <joint name="right_camera_optical_joint" type="fixed">
+    <parent link="right_camera_link"/>
+    <child link="right_camera_link_optical"/>
+    <origin xyz="0 0 0" rpy="${-pi/2} 0 ${-pi/2}" />
+  </joint>
+  <link name="right_camera_link_optical"></link>
+  <gazebo reference="right_camera_link">
+    <material>Gazebo/Green</material>
+    <sensor name="right_camera" type="camera">
+      <pose>0 0 0 0 0 0</pose>
+      <visualize>true</visualize>
+      <update_rate>10</update_rate>
+      <camera>
+        <horizontal_fov>1.089</horizontal_fov>
+        <image>
+          <format>R8G8B8</format>
+          <width>640</width>
+          <height>480</height>
+        </image>
+        <clip>
+          <near>0.005</near>
+          <far>20.0</far>
+        </clip>
+      </camera>
+      <plugin name="right_camera_controller" filename="libgazebo_ros_camera.so">
+        <image_topic_name>right_camera/image_raw</image_topic_name>
+        <frame_name>right_camera_link_optical</frame_name>
       </plugin>
     </sensor>

Commit message: updated robot model

File: ros/src/swarm_bot/description/camera.xacro (robot description, xacro)
@@ -5,5 +5,5 @@
     <parent link="chassis"/>
     <child link="left_camera_link"/>
-    <origin xyz="0.08 -0.05 0.025" rpy="0 0.005 0" />
+    <origin xyz="0.055 -0.0475 0.03" rpy="0 0.005 0" />
   </joint>
   <link name="left_camera_link">
@@ -11,5 +11,5 @@
     <visual>
       <geometry>
-        <box size="0.05 0.03 0.03" />
+        <box size="0.005 0.0254 0.0254 " />
       </geometry>
       <material name="blue"/>
@@ -50,5 +50,5 @@
     <parent link="chassis"/>
     <child link="right_camera_link"/>
-    <origin xyz="0.08 0.05 0.025" rpy="0 0.005 0" />
+    <origin xyz="0.055 0.0475 0.03" rpy="0 0.005 0" />
   </joint>
   <link name="right_camera_link">
@@ -56,5 +56,5 @@
     <visual>
       <geometry>
-        <box size="0.05 0.03 0.03" />
+        <box size="0.005 0.0254 0.0254" />
       </geometry>
       <material name="blue"/>

File: ros/src/swarm_bot/description/robot_core copy 2.xacro (robot description, xacro)
@@ -40,10 +40,7 @@
   <link name="chassis">
     <!-- Cylinder with r=120mm, h=50mm (ASSUMPTION) -->
-<!-- correct to a box with l = 114mm w = 68mm h = 76mm -->
-    <!-- Cylinder upwards length h = 15mm (incorrect) radius = 96mm somehwat correct-->
     <visual>
       <geometry>
-      <!-- length width heigh -->
-        <box size="0.1143 0.06858 0.076"/>
+        <cylinder length="0.05" radius="0.12"/>
       </geometry>
       <material name="white"/>
@@ -51,12 +48,12 @@
     <collision>
       <geometry>
-        <box size="0.1143 0.06858 0.076"/>
+        <cylinder length="0.05" radius="0.12"/>
       </geometry>
     </collision>
     <!-- Mass=0.5kg (ASSUMPTION) -->
-  <xacro:inertial_box mass="0.5" x="0.5" y="0.25" z="0.15">
-        <!-- Not sure if this is correct -->
-            <origin xyz="0 0 0.025" rpy="0 0 0"/>
-        </xacro:inertial_box>
+    <xacro:inertial_cylinder mass="0.5" length="0.05" radius="0.12">
+      <!-- Not sure if this is correct -->
+      <origin xyz="0 0 0.025" rpy="0 0 0"/>
+    </xacro:inertial_cylinder>
   </link>
   <gazebo reference="chassis">
@@ -67,5 +64,5 @@
     <parent link="base_link"/>
     <child link="left_wheel"/>
-    <origin xyz=".055 0.0375 0" rpy="-${pi/2} 0 0"/>
+    <origin xyz="0 0.1 0" rpy="-${pi/2} 0 0"/>
     <axis xyz="0 0 1"/>
   </joint>
@@ -95,5 +92,5 @@
     <parent link="base_link"/>
     <child link="right_wheel"/>
-    <origin xyz="0.055 -0.0375 0" rpy="${pi/2} 0 0"/>
+    <origin xyz="0 -0.10 0" rpy="${pi/2} 0 0"/>
     <axis xyz="0 0 -1"/>
   </joint>
@@ -124,5 +121,5 @@
 	<parent link="chassis"/>
 	<child link="caster_wheel"/>
-	<origin xyz="-.03125 0 -0.03"/>
+	<origin xyz="-0.0875 0 -0.03"/>
   </joint>
   <link name="caster_wheel">
@@ -150,3 +147,31 @@
 	<mu2>0.001</mu2>
   </gazebo>
-  </robot>
+  <joint name="front_caster_wheel_joint" type="fixed">
+    <parent link="chassis"/>
+    <child link="caster_wheel_2"/>
+    <origin xyz="0.0875 0 -0.03"/>
+  </joint>
+  <link name="caster_wheel_2">
+    <!-- Sphere with r=25mm (ASSUMPTION) -->
+    <visual>
+      <geometry>
+        <sphere radius="0.025"/>
+      </geometry>
+      <material name="red"/>
+    </visual>
+    <collision>
+      <geometry>
+        <sphere radius="0.025"/>
+      </geometry>
+    </collision>
+    <!-- Mass=0.1kg (ASSUMPTION) -->
+    <xacro:inertial_sphere mass="0.1" radius="0.025">
+      <origin xyz="0 0 0" rpy="0 0 0"/>
+    </xacro:inertial_sphere>
+  </link>
+  <gazebo reference="caster_wheel_2">
+    <material>Gazebo/Red</material>
+    <mu1>0.001</mu1>
+    <mu2>0.001</mu2>
+  </gazebo>
+</robot>

File: ros/src/swarm_bot/description/robot_core copy.xacro (robot description, xacro)
@@ -36,14 +36,11 @@
     <parent link="base_link"/>
     <child link="chassis"/>
-    <origin xyz="0 0 0.025" />
+    <origin xyz="0 0 0.025"/>
   </joint>
   <link name="chassis">
-    <!-- Cylinder with r=120mm, h=50mm (ASSUMPTION) -->
-<!-- correct to a box with l = 114mm w = 68mm h = 76mm -->
-    <!-- Cylinder upwards length h = 15mm (incorrect) radius = 96mm somehwat correct-->
+    <!-- Cylinder with r=46mm, length: 157 mm (laying down) (ASSUMPTION) -->
     <visual>
       <geometry>
-      <!-- length width heigh -->
-        <box size="0.1143 0.06858 0.076"/>
+        <cylinder length="0.157" radius="0.046"/>
       </geometry>
       <material name="white"/>
@@ -51,13 +48,14 @@
     <collision>
       <geometry>
-        <box size="0.1143 0.06858 0.076"/>
+        <cylinder length="0.157" radius="0.046"/>
       </geometry>
     </collision>
     <!-- Mass=0.5kg (ASSUMPTION) -->
-  <xacro:inertial_box mass="0.5" x="0.5" y="0.25" z="0.15">
-        <!-- Not sure if this is correct -->
-            <origin xyz="0 0 0.025" rpy="0 0 0"/>
-        </xacro:inertial_box>
+    <xacro:inertial_cylinder mass="0.5" length="0.05" radius="0.12">
+      <!-- Not sure if this is correct -->
+      <origin xyz="0 0 0.025" rpy="0 0 0"/>
+    </xacro:inertial_cylinder>
   </link>
+`
   <gazebo reference="chassis">
     <material>Gazebo/White</material>
@@ -67,5 +65,5 @@
     <parent link="base_link"/>
     <child link="left_wheel"/>
-    <origin xyz=".055 0.0375 0" rpy="-${pi/2} 0 0"/>
+    <origin xyz="0 0.1 0" rpy="-${pi/2} 0 0"/>
     <axis xyz="0 0 1"/>
   </joint>
@@ -95,5 +93,5 @@
     <parent link="base_link"/>
     <child link="right_wheel"/>
-    <origin xyz="0.055 -0.0375 0" rpy="${pi/2} 0 0"/>
+    <origin xyz="0 -0.10 0" rpy="${pi/2} 0 0"/>
     <axis xyz="0 0 -1"/>
   </joint>
@@ -124,5 +122,5 @@
 	<parent link="chassis"/>
 	<child link="caster_wheel"/>
-	<origin xyz="-.03125 0 -0.03"/>
+	<origin xyz="-0.0875 0 -0.03"/>
   </joint>
   <link name="caster_wheel">
@@ -150,3 +148,31 @@
 	<mu2>0.001</mu2>
   </gazebo>
-  </robot>
+  <joint name="front_caster_wheel_joint" type="fixed">
+    <parent link="chassis"/>
+    <child link="caster_wheel_2"/>
+    <origin xyz="0.0875 0 -0.03"/>
+  </joint>
+  <link name="caster_wheel_2">
+    <!-- Sphere with r=25mm (ASSUMPTION) -->
+    <visual>
+      <geometry>
+        <sphere radius="0.025"/>
+      </geometry>
+      <material name="red"/>
+    </visual>
+    <collision>
+      <geometry>
+        <sphere radius="0.025"/>
+      </geometry>
+    </collision>
+    <!-- Mass=0.1kg (ASSUMPTION) -->
+    <xacro:inertial_sphere mass="0.1" radius="0.025">
+      <origin xyz="0 0 0" rpy="0 0 0"/>
+    </xacro:inertial_sphere>
+  </link>
+  <gazebo reference="caster_wheel_2">
+    <material>Gazebo/Red</material>
+    <mu1>0.001</mu1>
+    <mu2>0.001</mu2>
+  </gazebo>
+</robot>

Commit message: working model

File: ros/src/swarm_bot/description/camera.xacro (robot description, xacro)
@@ -11,5 +11,5 @@
     <visual>
       <geometry>
-        <box size="0.005 0.0254 0.0254 " />
+        <box size="0.005 0.0154 0.0254 " />
       </geometry>
       <material name="blue"/>
