Commit message: nav kinda works, moving to aslam

File: ros/src/swarm_bot/description/lidar.xacro (robot description, xacro)
@@ -29,5 +29,5 @@
                 </scan>
                 <range>
-                    <min>0.3</min>
+                    <min>0.1</min>
                     <max>12</max>
                 </range>

File: ros/src/swarm_bot/description/robot_core.xacro (robot description, xacro)
@@ -64,5 +64,5 @@
     <parent link="base_link"/>
     <child link="left_wheel"/>
-    <origin xyz="0 0.122 0" rpy="-${pi/2} 0 0"/>
+    <origin xyz="0 0.1 0" rpy="-${pi/2} 0 0"/>
     <axis xyz="0 0 1"/>
   </joint>
@@ -92,5 +92,5 @@
     <parent link="base_link"/>
     <child link="right_wheel"/>
-    <origin xyz="0 -0.122 0" rpy="${pi/2} 0 0"/>
+    <origin xyz="0 -0.10 0" rpy="${pi/2} 0 0"/>
     <axis xyz="0 0 -1"/>
   </joint>
@@ -118,10 +118,39 @@
   <!-- CASTER WHEEL LINK -->
   <!-- Frictionless ball that does not rotate -->
-  <joint name="caster_wheel_joint" type="fixed">
-    <parent link="chassis"/>
-    <child link="caster_wheel"/>
-    <origin xyz="-0.0875 0 -0.03"/>
+   <joint name="caster_wheel_joint" type="fixed">
+	<parent link="chassis"/>
+	<child link="caster_wheel"/>
+	<origin xyz="-0.0875 0 -0.03"/>
   </joint>
   <link name="caster_wheel">
+	<!-- Sphere with r=25mm (ASSUMPTION) -->
+	<visual>
+  	<geometry>
+    	<sphere radius="0.025"/>
+  	</geometry>
+  	<material name="blue"/>
+	</visual>
+	<collision>
+  	<geometry>
+    	<sphere radius="0.025"/>
+  	</geometry>
+	</collision>
+	<!-- Mass=0.1kg (ASSUMPTION) -->
+	<xacro:inertial_sphere mass="0.1" radius="0.025">
+  	<origin xyz="0 0 0" rpy="0 0 0"/>
+	</xacro:inertial_sphere>
+  </link>
+  <!-- No friction -->
+  <gazebo reference="caster_wheel">
+	<material>Gazebo/Blue</material>
+	<mu1>0.001</mu1>
+	<mu2>0.001</mu2>
+  </gazebo>
+  <joint name="front_caster_wheel_joint" type="fixed">
+    <parent link="chassis"/>
+    <child link="caster_wheel_2"/>
+    <origin xyz="0.0875 0 -0.03"/>
+  </joint>
+  <link name="caster_wheel_2">
     <!-- Sphere with r=25mm (ASSUMPTION) -->
     <visual>
@@ -141,6 +170,5 @@
     </xacro:inertial_sphere>
   </link>
-  <!-- No friction -->
-  <gazebo reference="caster_wheel">
+  <gazebo reference="caster_wheel_2">
     <material>Gazebo/Red</material>
     <mu1>0.001</mu1>

Commit message: updated readme

File: ros/src/swarm_bot/description/lidar.xacro (robot description, xacro)
@@ -4,5 +4,5 @@
         <parent link="chassis"/>
         <child link="laser_frame"/>
-        <origin xyz="0.0 0.0 0.04" rpy="0 0 0"/>
+        <origin xyz="0.0 0 0.02" rpy="0 0 0"/>
     </joint>
     <link name="laser_frame">
@@ -13,4 +13,19 @@
             <material name="black"/>
         </visual>
+        <visual>
+            <origin xyz="0 0 -0.05"/>
+            <geometry>
+                <cylinder radius="0.01" length="0.1"/>
+            </geometry>
+            <material name="black"/>
+        </visual>
+        <collision>
+            <geometry>
+                <cylinder radius="0.05" length="0.04"/>
+            </geometry>
+        </collision>
+        <xacro:inertial_cylinder mass="0.1" length="0.04" radius="0.05">
+            <origin xyz="0 0 0" rpy="0 0 0"/>
+        </xacro:inertial_cylinder>
     </link>
     <gazebo reference="laser_frame">
@@ -18,5 +33,5 @@
         <sensor name="laser" type="ray">
             <pose> 0 0 0 0 0 0 </pose>
-            <visualize>true</visualize>
+            <visualize>false</visualize>
             <update_rate>10</update_rate>
             <ray>
@@ -29,5 +44,5 @@
                 </scan>
                 <range>
-                    <min>0.1</min>
+                    <min>0.3</min>
                     <max>12</max>
                 </range>

File: ros/src/swarm_bot/description/robot.urdf.xacro (robot description, xacro)
@@ -3,4 +3,5 @@
 <!-- ROS2 control is definitely better for the real robot but can be a little funkier in Gazebo -->
   <xacro:arg name="use_ros2_control" default="true" />
+  <xacro:arg name="sim_mode" default="false"/>
   <xacro:include filename="robot_core.xacro" />
   <xacro:if value="$(arg use_ros2_control)">

Commit message: performed some optimizations for aslam

File: ros/src/swarm_bot/description/lidar.xacro (robot description, xacro)
@@ -33,5 +33,5 @@
         <sensor name="laser" type="ray">
             <pose> 0 0 0 0 0 0 </pose>
-            <visualize>false</visualize>
+            <visualize>true</visualize>
             <update_rate>10</update_rate>
             <ray>
@@ -44,5 +44,5 @@
                 </scan>
                 <range>
-                    <min>0.3</min>
+                    <min>0.13</min>
                     <max>12</max>
                 </range>

File: ros/src/swarm_bot/description/robot_core.xacro (robot description, xacro)
@@ -40,10 +40,7 @@
   <link name="chassis">
     <!-- Cylinder with r=120mm, h=50mm (ASSUMPTION) -->
-<!-- correct to a box with l = 114mm w = 68mm h = 76mm -->
-    <!-- Cylinder upwards length h = 15mm (incorrect) radius = 96mm somehwat correct-->
     <visual>
       <geometry>
-      <!-- length width heigh -->
-        <box size="0.1143 0.06858 0.076"/>
+        <cylinder length="0.05" radius="0.12"/>
       </geometry>
       <material name="white"/>
@@ -51,12 +48,12 @@
     <collision>
       <geometry>
-        <box size="0.1143 0.06858 0.076"/>
+        <cylinder length="0.05" radius="0.12"/>
       </geometry>
     </collision>
     <!-- Mass=0.5kg (ASSUMPTION) -->
-  <xacro:inertial_box mass="0.5" x="0.5" y="0.25" z="0.15">
-        <!-- Not sure if this is correct -->
-            <origin xyz="0 0 0.025" rpy="0 0 0"/>
-        </xacro:inertial_box>
+    <xacro:inertial_cylinder mass="0.5" length="0.05" radius="0.12">
+      <!-- Not sure if this is correct -->
+      <origin xyz="0 0 0.025" rpy="0 0 0"/>
+    </xacro:inertial_cylinder>
   </link>
   <gazebo reference="chassis">
@@ -67,5 +64,5 @@
     <parent link="base_link"/>
     <child link="left_wheel"/>
-    <origin xyz=".055 0.0375 0" rpy="-${pi/2} 0 0"/>
+    <origin xyz="0 0.1 0" rpy="-${pi/2} 0 0"/>
     <axis xyz="0 0 1"/>
   </joint>
@@ -95,5 +92,5 @@
     <parent link="base_link"/>
     <child link="right_wheel"/>
-    <origin xyz="0.055 -0.0375 0" rpy="${pi/2} 0 0"/>
+    <origin xyz="0 -0.10 0" rpy="${pi/2} 0 0"/>
     <axis xyz="0 0 -1"/>
   </joint>
@@ -124,5 +121,5 @@
 	<parent link="chassis"/>
 	<child link="caster_wheel"/>
-	<origin xyz="-.03125 0 -0.03"/>
+	<origin xyz="-0.0875 0 -0.03"/>
   </joint>
   <link name="caster_wheel">
@@ -150,3 +147,31 @@
 	<mu2>0.001</mu2>
   </gazebo>
-  </robot>
+  <joint name="front_caster_wheel_joint" type="fixed">
+    <parent link="chassis"/>
+    <child link="caster_wheel_2"/>
+    <origin xyz="0.0875 0 -0.03"/>
+  </joint>
+  <link name="caster_wheel_2">
+    <!-- Sphere with r=25mm (ASSUMPTION) -->
+    <visual>
+      <geometry>
+        <sphere radius="0.025"/>
+      </geometry>
+      <material name="red"/>
+    </visual>
+    <collision>
+      <geometry>
+        <sphere radius="0.025"/>
+      </geometry>
+    </collision>
+    <!-- Mass=0.1kg (ASSUMPTION) -->
+    <xacro:inertial_sphere mass="0.1" radius="0.025">
+      <origin xyz="0 0 0" rpy="0 0 0"/>
+    </xacro:inertial_sphere>
+  </link>
+  <gazebo reference="caster_wheel_2">
+    <material>Gazebo/Red</material>
+    <mu1>0.001</mu1>
+    <mu2>0.001</mu2>
+  </gazebo>
+</robot>

Commit message: more work can be done but good enuf for now

File: ros/src/swarm_bot/description/lidar.xacro (robot description, xacro)
@@ -4,5 +4,5 @@
         <parent link="chassis"/>
         <child link="laser_frame"/>
-        <origin xyz="0.0 0 0.02" rpy="0 0 0"/>
+        <origin xyz="0.0 0 0.04" rpy="0 0 0"/>
     </joint>
     <link name="laser_frame">
@@ -44,5 +44,5 @@
                 </scan>
                 <range>
-                    <min>0.13</min>
+                    <min>0.10</min>
                     <max>12</max>
                 </range>
